Commit message: 完成sdk导入

File: src/hand_test/hand_description/urdf/omnihand_left.urdf (robot description, URDF)
Before this commit: robot omnihand, 24 links, 23 joints
Joints:
- joint L_index_dip_joint: limit lower=0 upper=1.8325957145940461 effort=1.764 velocity=0.308 -> lower=0 upper=2.03 effort=1.764 velocity=0.308; mimic joint=L_index_pip_joint multiplier=1.097 offset=0 -> joint=L_index_pip_joint multiplier=1.29 offset=0
- joint L_middle_dip_joint: limit lower=0 upper=1.8325957145940461 effort=1.764 velocity=0.308 -> lower=0 upper=2.03 effort=1.764 velocity=0.308; mimic joint=L_middle_pip_joint multiplier=1.097 offset=0 -> joint=L_middle_pip_joint multiplier=1.29 offset=0
- joint L_pinky_dip_joint: limit lower=0 upper=1.8325957145940461 effort=1.764 velocity=0.308 -> lower=0 upper=2.03 effort=1.764 velocity=0.308; mimic joint=L_pinky_pip_joint multiplier=1.097 offset=0 -> joint=L_pinky_pip_joint multiplier=1.29 offset=0
- joint L_ring_dip_joint: limit lower=0 upper=1.8325957145940461 effort=1.764 velocity=0.308 -> lower=0 upper=2.03 effort=1.764 velocity=0.308; mimic joint=L_ring_pip_joint multiplier=1.097 offset=0 -> joint=L_ring_pip_joint multiplier=1.29 offset=0
- joint L_thumb_dip_joint: limit lower=-1.1344640137963142 upper=0 effort=1.764 velocity=0.308 -> lower=-1.22 upper=0 effort=1.764 velocity=0.308; mimic joint=L_thumb_mcp_joint multiplier=1.3 offset=0 -> joint=L_thumb_mcp_joint multiplier=1.42 offset=0
- joint L_thumb_pip_joint: limit lower=-1.1384310735347046 upper=0 effort=1.764 velocity=0.308 -> lower=-1.14 upper=0 effort=1.764 velocity=0.308
